File: Dyna-Comp-606-5001-KiCad/Dyna-Comp-606-5001-KiCad.kicad_sch (KiCad schematic)
At the start: 97 parts, among them J1 Conn_01x05, J2 Conn_01x05, J3 Conn_01x06, Q1 2N3904, Q2 MPSU51, Q3 2N6543, Q4 2N3904, Q5 SCR1603, X1 0.1µF X, X2 0.1µF X

Commit message: Updated schematic title to include Apple part number
Other:
- title: Apple ][ DynaComp 606-5001 Power Supply 110v -> Apple ][ 605-5703 (DynaComp 606-5001) Power Supply 110v
Changed lines of the file:
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@@
 	(paper "A3")
 	(title_block
-		(title "Apple ][ DynaComp 606-5001 Power Supply 110v")
+		(title "Apple ][ 605-5703 (DynaComp 606-5001) Power Supply 110v")
 		(date "2025-10-12")
 		(rev "1")
