File: Dyna-Comp-606-5001-KiCad/Dyna-Comp-606-5001-KiCad.kicad_sch (KiCad schematic)
At the start: 97 parts, among them J1 Conn_01x05, J2 Conn_01x05, J3 Conn_01x06, Q1 2N3904, Q2 MPSU51, Q3 2N6543, Q4 2N3904, Q5 SCR1603, X1 0.1µF X, X2 0.1µF X

Commit message: V2, corrections, IEC filter, PCB layout
Parts:
- removed J1, J2: Conn_01x05, symbol Connector_Generic:Conn_01x05
- removed J3: Conn_01x06, symbol Connector_Generic:Conn_01x06
- removed PRIM5: Conn_01x01_Pin, symbol Connector:Conn_01x01_Pin
- removed TRW1, TRW2, TRW3, TRW4, TRW5, TRW6, TRW7, TRW_BL, TRW_WH: DynaCompTransformerWinding, symbol MyDynaCompLibrary:DynaComp_Transformer_Winding
- added J1001, J1002, J1003, J1004, J1005, J1006, J1007, J1008: Conn_01x01, Connector_Wire:SolderWire-0.25sqmm_1x01_D0.65mm_OD1.7mm, symbol Connector_Generic:Conn_01x01
- added T1001: Transformer_DynaComp, Transformer_THT:Transformer_EPCOS_B66359J1014T_Vertical, symbol Device:Transformer_1P_1S
- C1, C2: footprint (none) -> Capacitor_THT:CP_Radial_D10.0mm_P7.50mm
- C10, C12, C17, C18, C19, C20, C66: footprint (none) -> Capacitor_THT:CP_Radial_Tantal_D4.5mm_P5.00mm
- C11: value ???? -> C; footprint (none) -> Capacitor_THT:CP_Radial_Tantal_D4.5mm_P5.00mm; now not fitted
- C13: renamed from C12B; value **** -> C; footprint (none) -> Capacitor_THT:CP_Radial_Tantal_D4.5mm_P5.00mm
- C14: renamed from C13; footprint (none) -> Capacitor_THT:CP_Radial_Tantal_D4.5mm_P5.00mm
- C15: renamed from C14; footprint (none) -> Capacitor_THT:CP_Radial_Tantal_D4.5mm_P5.00mm
- C16: value C_Polarized -> C; footprint (none) -> Capacitor_THT:CP_Axial_L11.0mm_D5.0mm_P18.00mm_Horizontal
- C21: footprint (none) -> Capacitor_THT:C_Disc_D10.5mm_W5.0mm_P10.00mm
- C23, C77: footprint (none) -> Capacitor_THT:C_Rect_L11.0mm_W2.8mm_P10.00mm_MKT
- C3: value ???? -> C; now not fitted
- C4: footprint (none) -> Capacitor_THT:C_Disc_D4.3mm_W1.9mm_P5.00mm
- C5: footprint (none) -> Capacitor_THT:C_Axial_L17.0mm_D6.5mm_P25.00mm_Horizontal
- C6, C7: footprint (none) -> -my-footprints:-CP_Axial_P20.5mm_Horizontal
- C8: footprint (none) -> Capacitor_THT:C_Disc_D10.0mm_W2.5mm_P5.00mm
- CR10, CR2: footprint Diode_THT:D_DO-41_SOD81_P10.16mm_Horizontal -> Diode_THT:D_DO-34_SOD68_P12.70mm_Horizontal
- CR11, CR15, CR16, CR17, CR18, CR3, CR6, CR7, CR9: footprint (none) -> Diode_THT:D_DO-34_SOD68_P12.70mm_Horizontal
- CR12, CR13, CR14: value D_Small -> D; footprint (none) -> -my-footprints:-D_P10mm_Vertical_CathodeUp-Heatsink; symbol Device:D_Small -> Device:D
- CR19: footprint (none) -> Diode_THT:D_DO-34_SOD68_P10.16mm_Horizontal
- CR20, CR5: footprint (none) -> Diode_THT:D_A-405_P12.70mm_Horizontal
- FU1: footprint (none) -> Fuse:Fuse_SunFuse-6HP
- L1, L2, L3, L4: value ~ -> (none); footprint (none) -> -my-footprints:-L_Axial_P9mm
- L101, L102: footprint (none) -> -my-footprints:-L_Toroid_Vertical_P8.40mm
- Q1, Q4: footprint Package_TO_SOT_THT:TO-92_Inline -> -my-footprints:-TO-92_Wide-pin2-fwd
- Q2, Q5: footprint (none) -> Package_TO_SOT_THT:TO-220F-3_Vertical
- R10, R11, R12, R13, R14, R15, R17, R18, R2, R20, R21, R22, R23, R24, R25, R26, R27, R3, R4, R5, R6, R8, R9: footprint (none) -> -my-footprints:-R_Axial_P12.70mm_Horizontal
- R16: footprint (none) -> Potentiometer_THT:Potentiometer_Runtron_RM-063_Horizontal
- R19: footprint (none) -> Resistor_THT:R_Axial_DIN0207_L6.3mm_D2.5mm_P10.16mm_Horizontal
- TH1: footprint (none) -> Resistor_THT:R_Axial_DIN0204_L3.6mm_D1.6mm_P5.08mm_Horizontal
- X1, X2: footprint (none) -> Capacitor_THT:C_Rect_L16.5mm_W4.9mm_P15.00mm_MKT
- renumbered AR1 to AR1_1, AR1 to AR1_2, AR1 to AR1_3
Connections:
- net +12V: now also AR1_2.1, J1001.1 (ORG/WHT)
- net +5V: now also J1002.1 (ORG)
- net -12V: now also J1006.1 (BLU/WHT)
- net -5V: now also J1005.1 (BLU)
- net NEUT: now also J1007.1 (NEUT)
- net VAC: now also J1008.1 (LIVE)
- net AR1_4: now reaches AR1_3.1 (E), C6.2, C8.1, CR9.2 (A)
- net AR1_4: now also AR1_1.4, AR1_2.4
- net AR1_6: now reaches AR1_3.2 (B), C8.2
- net AR1_6: now also AR1_1.6, AR1_2.6
- net at C3.1, CR3.1 (K), FU1.2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: now also T1001.1 (CORE), T1001.3 (AA)
- net at CR16.1 (K): now also T1001.11 (SA)
- net at C10.2, C11.1, C12.1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: now also T1001.19 (SI)
- net at C23.1, C4.2, Q3.3 (C): now also T1001.4 (AB)
- net at C5.2, L102.2, X2.2: now also CR1.4; no longer CR1.2
- net at CR13.2 (A): now also T1001.18 (SH)
- net at CR3.2 (A), R23.1: now also T1001.6 (AD)
- net at C1.2, C2.2, C3.2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: now also Q3.0 (SH), T1001.2 (SH), T1001.5 (AC), T1001.7 (AE)
- net at CR14.2 (A): now also T1001.16 (SF)
- net at CR6.1 (K), R11.2: now also T1001.9 (AG)
- net at L101.2, X2.1: now also CR1.2; no longer CR1.4
- net at CR12.2 (A): now also T1001.20 (SJ)
- net at CR15.1 (K): now also T1001.13 (SC)
- net at R12.1, R13.1, R9.1: now also T1001.10 (AH)
- net AR1_5: now reaches AR1_3.3 (C), R14.2
- net AR1_5: now also AR1_1.5, AR1_2.5
- net at C14.2, C15.1, CR15.2 (A)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: now also T1001.12 (SB)
- net at R21.2: now also Q5.1 (G), R27.1; no longer Q5.3 (G)
- net AR1_2: now reaches AR1_2.2
- net AR1_2: now also AR1_1.2, R19.2
- net at R5.2: now also T1001.8 (AF)
- net GND (BLK) renamed GND
- net GND: now also Q5.3 (K), J1003.1 (BLK), J1004.1 (BLK), T1001.14 (SD), T1001.15 (SE), T1001.17 (SG); no longer Q5.1 (K), R27.1
- no-connect marks 1 -> 0
Other:
- note added: "BLUE"
- note added: "IEC LINE FILTER MODULE"
- note added: "Please check that you have the latest version of this schematic from: https://github.com/fredsa/apple-ii-dyna-comp-606-5001-power-supply Report any corrections to this schematic to: fredsa@gmail.com I've spent many hours recreating this schematic. If you found this schematic to be helful, please send me an email to let me know how it went."
- note added: "WHITE"
- note added: "diff"
- company: (none) -> Reverse-engineered by Fred Sauer in 2025.
- moved on the sheet: AR1_1, AR1_2, AR1_3, C1, C10, C12, C13, C14, C15, C16, C18, C19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

Commit message: Updated descriptions, publish PDF, SVG
Other:
- company: Reverse-engineered by Fred Sauer in 2025. -> Reverse-engineered by Fred Sauer in 2025, 2026.
- title: Apple ][ 605-5703 (DynaComp 606-5001) Power Supply 110v -> Apple II DynaComp Power Supply 110v
Changed lines of the file:
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@@
 	(paper "A3")
 	(title_block
-		(title "Apple ][ 605-5703 (DynaComp 606-5001) Power Supply 110v")
+		(title "Apple II DynaComp Power Supply 110v")
 		(date "2025-10-12")
-		(rev "2")
-		(company "Reverse-engineered by Fred Sauer in 2025.")
-		(comment 2 "U.S. Patent 4,130,862), except for differences indicated by dotted outline and 'diff' text.")
-		(comment 3 "The Apple II Circuit Description (reprint of Apple II Reference Manual 1981, see also")
-		(comment 4 "Part numbers and compontent layout match power supply schematic published in ")
+		(rev "3")
+		(company "Reverse-engineered by Fred Sauer in 2025, 2026.")
+		(comment 1 "U.S. Patent 4,130,862), except for differences indicated by dotted outlines marked 'diff'.")
+		(comment 2 "in The Apple II Circuit Description (reprint of Apple II Reference Manual 1981, see also")
+		(comment 3 "Part numbers and compontent layout updated to match power supply schematic published")
+		(comment 4 "DynaComp 606-5001, Apple part no. 605-5703")
 	)
 	(rectangle
